File: PCB/safe_chicks/safe_chicks.kicad_pcb (KiCad board)
At the start: 2 copper layers, 78 x 68 mm, 39 parts, among them J1 Conn_01x15, J10 Status LEDs, J11 UART, J12 SPI, J13 Conn_01x02, J2 Conn_01x15, J3 Battery Sensor, J4 Light Sensor, J5 Upper Switch, J6 Bottom Switch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

Commit message: update pcb
Parts:
- removed MH1, MH2, MH3, MH4: MountingHole_65mil, Arduino_MountingHole:MountingHole_65mil

Commit message: Created PCB
Parts:
- added G***: LOGO, LOGO, B.Cu at (133.0, 57.8)
Connections:
- J1 pad 13: /~{RESET} -> unconnected-(J1-Pin_13-Pad13)
- J2 pad 13: /~{RESET} -> unconnected-(J2-Pin_13-Pad13)
Routing:
- net /A4/SDA: track 31.1 -> 30.0 mm
- net /A1: track 56.8 -> 57.4 mm, vias 0 -> 1
- net /A0: track 36.2 -> 36.5 mm, vias 0 -> 1
- net /D13/SCK: track 42.7 -> 42.6 mm, vias 1 -> 3
Other:
- board text added: "3.3V"
- board text added: "5V"
- board text added: "BAT"
- board text added: "Dir"
- board text added: "GND"
- board text added: "Off"
- board text added: "On"
- board text added: "PWM (E1)"
- board text added: "RX"
- board text added: "TX"

Commit message: twerkt
Parts:
- added J14: Conn_01x02, Connector_PinHeader_2.54mm:PinHeader_1x02_P2.54mm_Vertical, F.Cu at (137.2, 67.9)
- added Q2: BS250, Package_TO_SOT_THT:TO-92_Inline, F.Cu at (141.5, 68.8)
- added R12: 10k, Resistor_THT:R_Axial_DIN0207_L6.3mm_D2.5mm_P10.16mm_Horizontal, F.Cu at (136.5, 59.5)
- added R13: 1k, Resistor_THT:R_Axial_DIN0207_L6.3mm_D2.5mm_P10.16mm_Horizontal, F.Cu at (136.5, 63.5)
- moved G*** 4.18 mm to (129.0, 56.5)
Routing:
- net Net-(Q2-G): track 0.00 -> 10.9 mm
- net Net-(J14-Pin_2): track 0.00 -> 4.93 mm
- net Net-(J14-Pin_1): track 0.00 -> 4.62 mm
Other:
- board text added: "In"
- board text added: "Out"
