File: PCB/safe_chicks/safe_chicks.kicad_sch (KiCad schematic)
At the start: 35 parts, among them J1 Conn_01x15, J10 Status LEDs, J11 UART, J12 SPI, J13 Conn_01x02, J2 Conn_01x15, J3 Battery Sensor, J4 Light Sensor, J5 Upper Switch, J6 Bottom Switch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

Commit message: Created PCB
Connections:
- net ~{RESET}: no longer names the net of J1.13 (Pin_13)
- net ~{RESET}: no longer J2.13 (Pin_13)
- no-connect marks 9 -> 10
Changed lines of the file:
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@@
+	)
+	(no_connect
+		(at 254 116.84)
 	)
 	(no_connect
@@
 		(effects
 			(font
-				(size 1.27 1.27)
-			)
-			(justify left bottom)
-		)
-	)
-	(label "~{RESET}"
-		(at 254 116.84 180)
-		(effects
-			(font
-				(size 1.27 1.27)
-			)
-			(justify right bottom)
-		)
-	)
-	(label "~{RESET}"
-		(at 200.66 116.84 0)
-		(effects
-			(font

Commit message: twerkt
Parts:
- added J14: Conn_01x02, Connector_PinHeader_2.54mm:PinHeader_1x02_P2.54mm_Vertical, symbol Connector_Generic:Conn_01x02
- added Q2: BS250, Package_TO_SOT_THT:TO-92_Inline, symbol Transistor_FET:BS250
- added R12: 10k, Resistor_THT:R_Axial_DIN0207_L6.3mm_D2.5mm_P10.16mm_Horizontal, symbol Device:R
- added R13: 1k, Resistor_THT:R_Axial_DIN0207_L6.3mm_D2.5mm_P10.16mm_Horizontal, symbol Device:R
- R6, R8: value 100k -> 10k
Connections:
- net +3V3: now also Q2.3 (S), R12.1
- new net: J14.2 (Pin_2), Q2.1 (D)
- new net: Q2.2 (G), R12.2, R13.2
- new net: J14.1 (Pin_1), R13.1
