File: V3/PCB/safe_chicks/safe_chicks.kicad_pcb (KiCad board)
At the start: 2 copper layers, 40 x 53 mm, 58 parts, among them J1 5V, J2 PGM, J3 Serial, J4 Buttons, J5 MOTOR, J6 Sensors, J8 Switches, J9 LED-Enable, SW1 Reset, U1 PIC18F2550-ISP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

Commit message: Move button pins so they can be used for interrupts
Connections:
- U1 pad 21: /U-SW -> /MU-BTN
- U1 pad 22: /B-SW -> /MD-BTN
- U1 pad 23: /MU-BTN -> /U-SW
- U1 pad 24: /MD-BTN -> /B-SW
Changed lines of the file:
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@@
 			(layers "*.Cu" "*.Mask")
 			(remove_unused_layers no)
-			(net 5 "/U-SW")
+			(net 8 "/MU-BTN")
 			(pinfunction "RB0/AN12/INT0/FLT0/SDI/SDA")
 			(pintype "bidirectional")
@@
 			(layers "*.Cu" "*.Mask")
 			(remove_unused_layers no)
-			(net 6 "/B-SW")
+			(net 9 "/MD-BTN")
 			(pinfunction "RB1/AN10/INT1/SCK/SCL")
 			(pintype "bidirectional")
@@
 			(layers "*.Cu" "*.Mask")
 			(remove_unused_layers no)
-			(net 8 "/MU-BTN")
+			(net 5 "/U-SW")
 			(pinfunction "RB2/AN8/INT2/VMO")
 			(pintype "bidirectional")
@@
 			(layers "*.Cu" "*.Mask")
 			(remove_unused_layers no)
-			(net 9 "/MD-BTN")
+			(net 6 "/B-SW")
 			(pinfunction "RB3/AN9/CCP2/VPO")
 			(pintype "bidirectional")
