File: V2/PCB/safe_chicks/safe_chicks.kicad_sch (KiCad schematic)
At the start: 56 parts, among them J1 5V, J10 B-SW, J11 PH-Sense, J12 MU-BTN, J13 MD-BTN, J2 PGM, J3 Serial, J5 MTR, J7 U-SW, J8 SP-Sense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

Commit message: More on PCB V2
Parts:
- removed J10: B-SW, symbol Connector_Generic:Conn_01x02
- removed J11: PH-Sense, symbol Connector_Generic:Conn_01x02
- removed J12: MU-BTN, symbol Connector_Generic:Conn_01x02
- removed J13: MD-BTN, symbol Connector_Generic:Conn_01x02
- removed J7: U-SW, symbol Connector_Generic:Conn_01x02
- removed J8: SP-Sense, symbol Connector_Generic:Conn_01x02
- added J4: Buttons, Connector_Molex:Molex_PicoBlade_53047-0410_1x04_P1.25mm_Vertical, symbol Connector_Generic:Conn_01x04
- added J6: Sensors, Connector_Molex:Molex_PicoBlade_53047-0410_1x04_P1.25mm_Vertical, symbol Connector_Generic:Conn_01x04
- added J8: Switches, Connector_Molex:Molex_PicoBlade_53047-0410_1x04_P1.25mm_Vertical, symbol Connector_Generic:Conn_01x04
- C1, C10, C11, C12, C2, C4, C6, C7, C8, C9: footprint (none) -> Capacitor_SMD:C_0603_1608Metric_Pad1.08x0.95mm_HandSolder
- C3, C5: footprint (none) -> Capacitor_Tantalum_SMD:CP_EIA-3216-10_Kemet-I_HandSolder
- D1: footprint (none) -> Diode_THT:D_DO-15_P10.16mm_Horizontal
- D2, D3, D4, D5, D6, D7: footprint (none) -> LED_SMD:LED_0603_1608Metric_Pad1.05x0.95mm_HandSolder
- H1, H2, H3, H4: footprint (none) -> MountingHole:MountingHole_3.2mm_M3_Pad_Via
- J1: footprint (none) -> TerminalBlock:TerminalBlock_bornier-2_P5.08mm
- J2, J5: footprint (none) -> Connector_PinHeader_2.54mm:PinHeader_1x06_P2.54mm_Vertical
- J3: footprint (none) -> Connector_Molex:Molex_PicoBlade_53047-0410_1x04_P1.25mm_Vertical
- J9: footprint (none) -> Connector_PinHeader_2.54mm:PinHeader_1x03_P2.54mm_Vertical
- R1, R10, R11, R12, R13, R14, R15, R16, R17, R18, R19, R2, R20, R3, R4, R6, R7, R8, R9: footprint (none) -> Resistor_SMD:R_0603_1608Metric_Pad0.98x0.95mm_HandSolder
- SW1: footprint (none) -> Button_Switch_THT:SW_PUSH_6mm_H4.3mm
- Y1: footprint (none) -> Crystal:Crystal_HC49-U_Vertical
Connections:
- net GND: now also J1.2 (Pin_2); no longer J1.1 (Pin_1)
- net PH-ADC: now also J6.4 (Pin_4)
- net SP+: now also J6.1 (Pin_1)
- net SP-: now also J6.2 (Pin_2)
- net VDD: now also J1.1 (Pin_1), J4.1 (Pin_1), J4.3 (Pin_3), J6.3 (Pin_3), J8.1 (Pin_1), J8.3 (Pin_3); no longer J1.2 (Pin_2)
- net BTN-UP: now reaches R17.2, R18.2
- net BTN-UP: now also J4.2 (Pin_2)
- net SW-Upper: now reaches R10.2, R6.2
- net SW-Upper: now also J8.2 (Pin_2)
- net BTN-DOWN: now reaches R19.2, R20.2
- net BTN-DOWN: now also J4.4 (Pin_4)
- net SW-Bottom: now reaches R11.2, R7.2
- net SW-Bottom: now also J8.4 (Pin_4)
Other:
- moved on the sheet: H1, J1

Commit message: FSM is working with buttons and motor runs
Parts:
- R2, R3: value 613k -> 316k
Changed lines of the file:
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@@
 			)
 		)
-		(property "Value" "613k"
+		(property "Value" "316k"
 			(at 245.11 43.18 90)
 			(effects
@@
 			)
 		)
-		(property "Value" "613k"
+		(property "Value" "316k"
 			(at 245.11 48.26 90)
 			(effects

Commit message: This works but sensors could be better
Other:
- note added: "Better to put the IC on the chip itself for more control (low power)"
- note added: "No cristal needed"
- note added: "Wrong RC4 and RC5 are input only"
Changed lines of the file:
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@@
+		)
+	)
+	(text "Better to put the\nIC on the chip itself\nfor more control\n(low power)"
+		(exclude_from_sim no)
+		(at 251.968 26.924 0)
+		(effects
+			(font
+				(size 1.27 1.27)
+				(color 255 0 0 1)
+			)
+			(justify right)
 		)
 	)
@@
 		)
 	)
+	(text "Wrong\nRC4 and RC5 are input only"
+		(exclude_from_sim no)
+		(at 114.3 51.054 0)
+		(effects
+			(font
+				(size 1.27 1.27)
+				(color 255 0 0 1)
+			)
+			(justify left)
+		)
+	)
+	(text "No cristal\nneeded"
+		(exclude_from_sim no)
+		(at 26.924 61.214 0)
+		(effects
+			(font
+				(size 1.27 1.27)
+				(color 255 0 0 1)
+			)
+			(justify right)
+		)
+	)

Commit message: I think we are ready
Other:
- note added: "Does not match reality any more RB0=BTN UP RB1=BTN DWN RB2=x RB3=Limit switch"
Changed lines of the file:
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@@
+		)
+	)
+	(text "Does not match\nreality any more\nRB0=BTN UP\nRB1=BTN DWN\nRB2=x\nRB3=Limit switch"
+		(exclude_from_sim no)
+		(at 30.226 72.644 0)
+		(effects
+			(font
+				(size 1.27 1.27)
+				(color 255 0 0 1)
+			)
+			(justify right)
 		)
 	)

Commit message: Added parts to readme
Other:
- note added: "MOTOR DRIVER SKU:DRI0044 DFROBOT"
- note added: "These inputs are connected to the buttons to have input interrupts"
- note added: "This is now the limit switch"
Changed lines of the file:
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@@
+		)
+	)
+	(text "These inputs are connected to the buttons\nto have input interrupts"
+		(exclude_from_sim no)
+		(at 179.578 66.802 0)
+		(effects
+			(font
+				(size 1.27 1.27)
+				(color 255 0 0 1)
+			)
 		)
 	)
@@
 		)
 	)
+	(text "This is now the limit switch"
+		(exclude_from_sim no)
+		(at 188.722 132.08 0)
+		(effects
+			(font
+				(size 1.27 1.27)
+				(color 255 0 0 1)
+			)
+		)
+	)
 	(text "Wrong\nRC4 and RC5 are input only"
 		(exclude_from_sim no)
@@
 		)
 	)
+	(text "MOTOR DRIVER\nSKU:DRI0044\nDFROBOT"
+		(exclude_from_sim no)
+		(at 272.288 18.796 0)
+		(effects
+			(font
+				(size 1.27 1.27)
+			)
+		)
+	)
